File: Hardware/KiCAD/sa8x8-breakout/sa8x8-breakout.kicad_pcb (KiCad board)
At the start: 2 copper layers, 49.6 x 35.6 mm, 10 parts, among them J1 Conn_01x10, J2 Conn_01x10, J3 Conn_Coaxial, J4 Conn_01x07, J5 Conn_01x04, J6 Conn_01x07

Commit message: chore: move KiCAD files into dedicated directory
Parts:
- added U1: SA868, sa8x8:G-NICERF_SA868, F.Cu at (150.4, 89.5)
