File: Hardware/KiCAD/spur-demo/display.kicad_sch (KiCad schematic)
At the start: 9 parts

Commit message: feat: begin footprint assignment, unify +3.3V PWRREFs
Parts:
- C19, C20, C21, C22: footprint (none) -> Capacitor_SMD:C_0603_1608Metric_Pad1.08x0.95mm_HandSolder
- R36: footprint (none) -> Resistor_SMD:R_0603_1608Metric
Changed lines of the file:
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@@
 			)
 		)
-		(property "Footprint" ""
+		(property "Footprint" "Capacitor_SMD:C_0603_1608Metric_Pad1.08x0.95mm_HandSolder"
 			(at 94.9452 34.29 0)
 			(effects
@@
 			)
 		)
-		(property "Footprint" ""
+		(property "Footprint" "Capacitor_SMD:C_0603_1608Metric_Pad1.08x0.95mm_HandSolder"
 			(at 50.8 33.3248 0)
 			(effects
@@
 			)
 		)
-		(property "Footprint" ""
+		(property "Footprint" "Capacitor_SMD:C_0603_1608Metric_Pad1.08x0.95mm_HandSolder"
 			(at 50.8 42.8752 0)
 			(effects
@@
 			)
 		)
-		(property "Footprint" ""
+		(property "Footprint" "Capacitor_SMD:C_0603_1608Metric_Pad1.08x0.95mm_HandSolder"
 			(at 65.7352 113.03 0)
 			(effects
@@
 			)
 		)
-		(property "Footprint" ""
+		(property "Footprint" "Resistor_SMD:R_0603_1608Metric"
 			(at 53.086 108.966 90)
 			(effects

Commit message: feat: assign solder jumper footprints, begin testpoints
Parts:
- added R40: 10k, Resistor_SMD:R_0603_1608Metric, symbol Device:R_US
- added TP1, TP2, TP3, TP4, TP5: TestPoint, TestPoint:TestPoint_Loop_D2.54mm_Drill1.5mm_Beaded, symbol Connector:TestPoint
- JP10, JP8, JP9: footprint (none) -> Jumper:SolderJumper-3_P1.3mm_Bridged12_RoundedPad1.0x1.5mm_NumberLabels
Connections:
- net +3.3V: now also R40.2
- net D0: now also TP4.1
- net D1: now also TP5.1
- net D/~{C}: now also TP2.1
- net ~{CS}: now also TP3.1
- net ~{RES}: now also R40.1, TP1.1
Other:
- moved on the sheet: C19, C20, C21, C22, DS1, JP10, JP8, JP9, R36

Commit message: feat: squash recaptured schematics and footprint reassignments
Parts:
- C19, C20, C21, C22, DS1, JP10, JP8, JP9, R36, R40, TP1, TP2, TP3, TP4, TP5: now not fitted
