File: Hardware/KiCAD/spur-demo/audio_subsystem.kicad_sch (KiCad schematic)
At the start: 16 parts, among them U3 MAX98357A, U4 LM393

Commit message: feat: configuration for audio amp through solder jumpers with set defaults
Parts:
- added JP1: GAIN_{LOGIC}, symbol Jumper:SolderJumper_3_Open
- added JP2: GAIN_{R}, symbol Jumper:SolderJumper_3_Open
- added JP3: CH_LEFT, symbol Jumper:SolderJumper_2_Open
- added JP4: CH_MIX, symbol Jumper:SolderJumper_2_Open
- added JP5: CH_RIGHT, symbol Jumper:SolderJumper_2_Open
- added JP6: Driver, symbol Jumper:SolderJumper_3_Bridged12
- added R13: 100k, symbol Device:R_US
- added R14: 330k, symbol Device:R_US
- added R37: 2k, symbol Device:R_US
- R28: now fitted
- R29: value 100k 5% -> 680k; now fitted
Connections:
- net +3.3V: now also JP1.1 (A), JP6.1 (A); no longer MK1.1 (-), R28.1, R28.2, R29.1, R29.2, R30.2, R35.2, U3.11 (GND), U3.15 (GND), U3.2 (GAIN_SLOT), U3.3 (GND), U4.4 (V-), VR1.1 (CCW)
- net ~{AMP_SD}: now also R29.2, JP3.1 (A), R14.1; no longer U3.4 (~{SD_MODE})
- new net: JP6.2 (C), R37.1
- new net: JP4.1 (A), R29.1
- new net: JP1.2 (C), JP2.1 (A), R28.1
- new net: JP5.1 (A), R14.2
- new net: JP2.3 (B), R28.2
- new net GAIN_SLOT: JP2.2 (C), U3.2 (GAIN_SLOT)
- new net GND: JP1.3 (B), MK1.1 (-), R13.1, R30.2, R35.2, U3.11 (GND), U3.15 (GND), U3.3 (GND), U4.4 (V-), VR1.1 (CCW)
- new net ~{SD_MODE}: JP3.2 (B), JP4.2 (B), JP5.2 (B), JP6.3 (B), R13.2, R37.2, U3.4 (~{SD_MODE})
- no-connect marks 4 -> 3
Other:
- note added: "CHANNEL MODE SELECT: MIX (MONO) SD < 0.16V = Turn off amplifier (GND) SD 0.16V to 0.77V = Output mix channel (R_{large} pullup) SD < 0.16V = Output right channel (R_{small} pullup) SD > 1.4V = Output left channel (2k pullup)"
- note added: "Open-Drain Driver: JP6 1:2 Push-Pull Driver: JP6 3:2"
- note added: "R_{small} = 94.0 * V_{DDIO} - 100 R_{large} = 222.2 * V_{DDIO} - 100 V_{DDIO} = 3.3V R_{small} = 210.2k, placed 330k R_{large} = 634k, placed 680k"
- note removed: "SD SELECT: SD < 0.16V = Turn off amplifier (GND) SD 0.16V to 0.77V = Output mix channel (3.3V series 680k) SD < 0.16V = Output right channel (3.3V series 330k) SD > 1.4V = Output left channel (3.3V series 100k)"
- moved on the sheet: LS1, U3, VR1

Commit message: fix: set JP6 to use audio amp as mono
Parts:
- JP4: symbol Jumper:SolderJumper_2_Open -> Jumper:SolderJumper_2_Bridged
Changed lines of the file:
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@@
 	)
 	(symbol
-		(lib_id "Jumper:SolderJumper_2_Open")
+		(lib_id "Jumper:SolderJumper_2_Bridged")
 		(at 241.3 83.82 0)
 		(mirror x)
@@
 			)
 		)
-		(property "Description" "Solder Jumper, 2-pole, open"
+		(property "Description" "Solder Jumper, 2-pole, closed/bridged"
 			(at 241.3 83.82 0)
 			(effects

Commit message: fix: give mic level setpoint potentiometer a name
Parts:
- RV1: value R_Potentiometer_US -> Level setpoint
Other:
- moved on the sheet: U4C

Commit message: feat: begin footprint assignment, unify +3.3V PWRREFs
Parts:
- D3, D4: footprint (none) -> LED_SMD:LED_0603_1608Metric_Pad1.05x0.95mm_HandSolder
- LS1: footprint (none) -> Connector_JST:JST_XH_S2B-XH-A_1x02_P2.50mm_Horizontal
- MK1: footprint (none) -> Sensor_Audio:POM-2244P-C3310-2-R
- R13, R14, R28, R29, R30, R31, R32, R33, R34, R35, R37: footprint (none) -> Resistor_SMD:R_0603_1608Metric
- RV1: footprint (none) -> Potentiometer_SMD:Potentiometer_Bourns_3214W_Vertical
- U4: footprint (none) -> Package_SO:VSSOP-8_3x3mm_P0.65mm
Changed lines of the file:
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@@
 			)
 		)
-		(property "Footprint" ""
+		(property "Footprint" "LED_SMD:LED_0603_1608Metric_Pad1.05x0.95mm_HandSolder"
 			(at 57.15 107.95 0)
 			(effects
@@
 			)
 		)
-		(property "Footprint" ""
+		(property "Footprint" "LED_SMD:LED_0603_1608Metric_Pad1.05x0.95mm_HandSolder"
 			(at 57.15 97.79 0)
 			(effects
@@
 			)
 		)
-		(property "Footprint" ""
+		(property "Footprint" "Resistor_SMD:R_0603_1608Metric"
 			(at 46.736 98.806 90)
 			(effects
@@
 			)
 		)
-		(property "Footprint" ""
+		(property "Footprint" "Resistor_SMD:R_0603_1608Metric"
 			(at 249.174 100.076 90)
 			(effects
@@
 			)
 		)
-		(property "Footprint" ""
+		(property "Footprint" "Connector_JST:JST_XH_S2B-XH-A_1x02_P2.50mm_Horizontal"
 			(at 269.24 40.64 0)
 			(effects
@@
 			)
 		)
-		(property "Footprint" ""
+		(property "Footprint" "Package_SO:VSSOP-8_3x3mm_P0.65mm"
 			(at 41.91 60.96 0)
 			(effects
@@
 			)
 		)
-		(property "Footprint" ""
+		(property "Footprint" "Resistor_SMD:R_0603_1608Metric"
 			(at 60.706 36.576 90)
 			(effects
@@
 			)
 		)
-		(property "Footprint" ""
+		(property "Footprint" "Resistor_SMD:R_0603_1608Metric"
 			(at 46.736 108.966 90)
 			(effects
@@
 			)
 		)
-		(property "Footprint" ""
+		(property "Footprint" "Resistor_SMD:R_0603_1608Metric"
 			(at 60.706 78.486 90)
 			(effects
@@
 			)
 		)
-		(property "Footprint" ""
+		(property "Footprint" "Resistor_SMD:R_0603_1608Metric"
 			(at 228.346 84.836 90)
 			(effects
@@
 			)
 		)
-		(property "Footprint" ""
+		(property "Footprint" "Package_SO:VSSOP-8_3x3mm_P0.65mm"
 			(at 34.29 87.63 0)
 			(effects
@@
 			)
 		)
-		(property "Footprint" ""
+		(property "Footprint" "Resistor_SMD:R_0603_1608Metric"
 			(at 215.646 39.624 90)
 			(effects
@@
 			)
 		)
-		(property "Footprint" ""
+		(property "Footprint" "Resistor_SMD:R_0603_1608Metric"
 			(at 228.854 92.964 90)
 			(effects
@@
 			)
 		)
-		(property "Footprint" ""
+		(property "Footprint" "Package_SO:VSSOP-8_3x3mm_P0.65mm"
 			(at 78.74 38.1 0)
 			(effects
@@
 			)
 		)
-		(property "Footprint" ""
+		(property "Footprint" "Sensor_Audio:POM-2244P-C3310-2-R"
 			(at 41.91 26.67 90)
 			(effects
@@
 			)
 		)
-		(property "Footprint" ""
+		(property "Footprint" "Resistor_SMD:R_0603_1608Metric"
 			(at 25.146 36.576 90)
 			(effects
@@
 			)
 		)
-		(property "Footprint" ""
+		(property "Footprint" "Resistor_SMD:R_0603_1608Metric"
 			(at 225.044 146.304 90)
 			(effects
@@
 			)
 		)
-		(property "Footprint" ""
+		(property "Footprint" "Resistor_SMD:R_0603_1608Metric"
 			(at 50.546 42.164 90)
 			(effects
@@
 			)
 		)
-		(property "Footprint" ""
+		(property "Footprint" "Potentiometer_SMD:Potentiometer_Bourns_3214W_Vertical"
 			(at 60.96 48.26 0)
 			(effects

Commit message: feat: assign solder jumper footprints, begin testpoints
Parts:
- JP1, JP2: footprint (none) -> Jumper:SolderJumper-3_P1.3mm_Open_RoundedPad1.0x1.5mm_NumberLabels
- JP3, JP5: footprint (none) -> Jumper:SolderJumper-2_P1.3mm_Open_RoundedPad1.0x1.5mm
- JP4: footprint (none) -> Jumper:SolderJumper-2_P1.3mm_Bridged_Pad1.0x1.5mm
- JP6: footprint (none) -> Jumper:SolderJumper-3_P1.3mm_Bridged12_RoundedPad1.0x1.5mm_NumberLabels
- RV1: footprint Potentiometer_SMD:Potentiometer_Bourns_3214W_Vertical -> Potentiometer_SMD:Potentiometer_Bourns_3314G_Vertical
Changed lines of the file:
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@@
 			)
 		)
-		(property "Footprint" ""
+		(property "Footprint" "Jumper:SolderJumper-3_P1.3mm_Bridged12_RoundedPad1.0x1.5mm_NumberLabels"
 			(at 205.74 33.02 0)
 			(effects
@@
 			)
 		)
-		(property "Footprint" ""
+		(property "Footprint" "Jumper:SolderJumper-3_P1.3mm_Open_RoundedPad1.0x1.5mm_NumberLabels"
 			(at 212.09 147.32 0)
 			(effects
@@
 			)
 		)
-		(property "Footprint" ""
+		(property "Footprint" "Jumper:SolderJumper-2_P1.3mm_Bridged_Pad1.0x1.5mm"
 			(at 241.3 83.82 0)
 			(effects
@@
 			)
 		)
-		(property "Footprint" ""
+		(property "Footprint" "Jumper:SolderJumper-3_P1.3mm_Open_RoundedPad1.0x1.5mm_NumberLabels"
 			(at 231.14 139.7 0)
 			(effects
@@
 			)
 		)
-		(property "Footprint" ""
+		(property "Footprint" "Jumper:SolderJumper-2_P1.3mm_Open_RoundedPad1.0x1.5mm"
 			(at 241.3 73.66 0)
 			(effects
@@
 			)
 		)
-		(property "Footprint" ""
+		(property "Footprint" "Jumper:SolderJumper-2_P1.3mm_Open_RoundedPad1.0x1.5mm"
 			(at 241.3 93.98 0)
 			(effects
@@
 			)
 		)
-		(property "Footprint" "Potentiometer_SMD:Potentiometer_Bourns_3214W_Vertical"
+		(property "Footprint" "Potentiometer_SMD:Potentiometer_Bourns_3314G_Vertical"
 			(at 60.96 48.26 0)
 			(effects

Commit message: feat: establish microphone module footprint and header
Parts:
- added J4: VMA309 Module, spur-demo:VMA309, symbol Connector:Conn_01x04_Socket
Connections:
- net +3.3V: now also J4.2 (Pin_2)
- net GND: now also J4.3 (Pin_3)
- net MIC_OUT_A: now also J4.4 (Pin_4)
- net MIC_OUT_D: now also J4.1 (Pin_1)
Other:
- moved on the sheet: VR1

Commit message: feat: squash recaptured schematics and footprint reassignments
Parts:
- added J7: PAM8392A Module, spur-demo:PAM8392A, symbol Connector:Conn_01x05_Socket
- D3, D4, MK1, R30, R31, R32, R33, R34, R35, RV1, U4: now not fitted
Connections:
- net +3.3V: now also J7.4 (Pin_4); no longer VR1.4 (COM)
- net AF+: now also J7.1 (Pin_1)
- net AF-: now also J7.2 (Pin_2)
- net GND: now also J7.5 (Pin_5)
- net ~{AMP_SD}: now also J7.3 (Pin_3)
- new net +SYS: VR1.4 (COM)
Other:
- moved on the sheet: J4
