File: Hardware/KiCAD/spur-demo/computing_subsystem.kicad_sch (KiCad schematic)
At the start: 22 parts, among them J3 SD_Card, J8 1x15, J9 1x15, SW1 SW_Push, SW2 SW_Push, U2 ESP32-C3-WROOM-02

Commit message: feat: begin footprint assignment, unify +3.3V PWRREFs
Parts:
- C13, C14, C15, C16, C17: footprint Capacitor_SMD:C_0603_1608Metric -> Capacitor_SMD:C_0603_1608Metric_Pad1.08x0.95mm_HandSolder
Connections:
- net 3.3V renamed +3.3V
Changed lines of the file:
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@@
 			)
 		)
-		(property "Value" "3.3V"
+		(property "Value" "+3.3V"
 			(at 215.9 54.61 0)
 			(effects
@@
 			)
 		)
-		(property "Footprint" "Capacitor_SMD:C_0603_1608Metric"
+		(property "Footprint" "Capacitor_SMD:C_0603_1608Metric_Pad1.08x0.95mm_HandSolder"
 			(at 28.9052 58.42 0)
 			(effects
@@
 			)
 		)
-		(property "Footprint" "Capacitor_SMD:C_0603_1608Metric"
+		(property "Footprint" "Capacitor_SMD:C_0603_1608Metric_Pad1.08x0.95mm_HandSolder"
 			(at 53.0352 67.31 0)
 			(effects
@@
 			)
 		)
-		(property "Value" "3.3V"
+		(property "Value" "+3.3V"
 			(at 175.26 64.77 0)
 			(effects
@@
 			)
 		)
-		(property "Footprint" "Capacitor_SMD:C_0603_1608Metric"
+		(property "Footprint" "Capacitor_SMD:C_0603_1608Metric_Pad1.08x0.95mm_HandSolder"
 			(at 201.93 32.0548 0)
 			(effects
@@
 			)
 		)
-		(property "Footprint" "Capacitor_SMD:C_0603_1608Metric"
+		(property "Footprint" "Capacitor_SMD:C_0603_1608Metric_Pad1.08x0.95mm_HandSolder"
 			(at 38.4048 74.93 0)
 			(effects
@@
 			)
 		)
-		(property "Value" "3.3V"
+		(property "Value" "+3.3V"
 			(at 91.44 31.75 0)
 			(effects
@@
 			)
 		)
-		(property "Footprint" "Capacitor_SMD:C_0603_1608Metric"
+		(property "Footprint" "Capacitor_SMD:C_0603_1608Metric_Pad1.08x0.95mm_HandSolder"
 			(at 236.22 32.0548 0)
 			(effects
@@
 			)
 		)
-		(property "Value" "3.3V"
+		(property "Value" "+3.3V"
 			(at 229.87 118.11 0)
 			(effects
@@
 			)
 		)
-		(property "Value" "3.3V"
+		(property "Value" "+3.3V"
 			(at 278.13 17.78 0)
 			(effects

Commit message: chore: name boot and reset push buttons
Parts:
- SW1: value SW_Push -> BOOT
- SW2: value SW_Push -> RESET
Changed lines of the file:
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@@
 			)
 		)
-		(property "Value" "SW_Push"
+		(property "Value" "RESET"
 			(at 232.41 22.86 0)
 			(effects
@@
 			)
 		)
-		(property "Value" "SW_Push"
+		(property "Value" "BOOT"
 			(at 205.74 22.86 0)
 			(effects

Commit message: feat: squash recaptured schematics and footprint reassignments
Parts:
- removed C13: 1u, Capacitor_SMD:C_0603_1608Metric_Pad1.08x0.95mm_HandSolder, symbol Device:C
- removed C14: 10u, Capacitor_SMD:C_0603_1608Metric_Pad1.08x0.95mm_HandSolder, symbol Device:C
- removed C16: 0.1u, Capacitor_SMD:C_0603_1608Metric_Pad1.08x0.95mm_HandSolder, symbol Device:C
- removed R11: 10k, Resistor_SMD:R_0603_1608Metric, symbol Device:R_US
- removed U2: ESP32-C3-WROOM-02, PCM_Espressif:ESP32-C3-WROOM-02, symbol PCM_Espressif:ESP32-C3-WROOM-02
- added U5: XCVR_ESP32-C3-DEVKITM-1, spur-demo:XCVR_ESP32-C3-DEVKITM-1, symbol spur-demo:ESP32-C3-DEVKITM-1
- C15, C17, SW1, SW2: now not fitted; now left out of the parts list
- J8, J9: footprint Connector_PinHeader_2.54mm:PinHeader_1x15_P2.54mm_Vertical -> Connector_PinSocket_2.54mm:PinSocket_1x15_P2.54mm_Vertical
- R12: now left out of the parts list
Connections:
- net +3.3V: now also U5.2 (3V3), U5.3 (3V3)
- net +5V: now also U5.13 (5V), U5.14 (5V)
- net GND: now also J8.12 (Pin_12), J8.6 (Pin_6), J8.8 (Pin_8), J9.12 (Pin_12), J9.4 (Pin_4), J9.7 (Pin_7), U5.1 (GND), U5.12 (GND), U5.15 (GND), U5.16 (GND), U5.19 (GND), U5.24 (GND), U5.27 (GND), U5.30 (GND), U5.6 (GND), U5.8 (GND); no longer J8.10 (Pin_10), J8.5 (Pin_5), J9.11 (Pin_11), J9.14 (Pin_14), J9.6 (Pin_6), J9.8 (Pin_8)
- net GPIO0/ADC1_CH0: now also J8.9 (Pin_9), U5.9 (IO0); no longer J9.2 (Pin_2)
- net GPIO10: now also J8.11 (Pin_11), U5.11 (IO10); no longer J9.7 (Pin_7)
- net GPIO20/U0RXD: now also J9.3 (Pin_3), U5.28 (RX); no longer J9.9 (Pin_9)
- net GPIO21/U0TXD: now also J9.2 (Pin_2), U5.29 (TX); no longer J9.10 (Pin_10)
- net GPIO4/ADC1_CH4: now also J9.11 (Pin_11), U5.20 (IO4); no longer J8.6 (Pin_6)
- net GPIO5/ADC2_CH0: now also J9.10 (Pin_10), U5.21 (IO5); no longer J8.7 (Pin_7)
- net GPIO8: now also J9.6 (Pin_6), U5.25 (IO8); no longer J8.11 (Pin_11)
- net GPIO9: now also J9.5 (Pin_5), U5.26 (IO9); no longer J8.12 (Pin_12)
- net I2C0_SCL: now also J8.5 (Pin_5), U5.5 (IO3); no longer J9.5 (Pin_5)
- net I2C0_SDA: now also J8.10 (Pin_10), U5.10 (IO1); no longer J9.3 (Pin_3)
- net RST: now also J8.7 (Pin_7), U5.7 (RST); no longer J8.4 (Pin_4)
- net SPIM2_MISO: now also J8.4 (Pin_4), U5.4 (IO2); no longer J9.4 (Pin_4)
- net SPIM2_MOSI: now also J9.8 (Pin_8), U5.23 (IO7); no longer J8.9 (Pin_9)
- net SPIM2_SCLK: now also J9.9 (Pin_9), U5.22 (IO6); no longer J8.8 (Pin_8)
- net USB_DN: now also J9.13 (Pin_13), U5.18 (IO18); no longer J9.12 (Pin_12)
- net USB_DP: now also J9.14 (Pin_14), U5.17 (IO19); no longer J9.13 (Pin_13)
- net SD_DAT3 renamed ~{SD_CS}
