File: Hardware/KiCAD/spur-demo/keypad.kicad_sch (KiCad schematic)
At the start: 40 parts, among them SW10 *, SW11 4, SW12 5, SW13 6, SW14 0, SW15 7, SW16 8, SW17 9, SW18 #, SW19 PTT, SW20 LEFT, SW21 RIGHT, SW22 SK0, SW3 MENU, SW4 UP, SW5 DOWN, SW6 EXIT, SW7 1, SW8 2, SW9 3

Commit message: fix: remove node breaking col1 and row4 net resolution
Parts:
- renumbered D2:1 to D1:1, D2:2 to D1:2, D2:3 to D1:3, D1:2 to D1:4, D3:1 to D2:1, D3:2 to D2:2, D3:3 to D2:3, D1:3 to D2:4, D1:1 to D2:5, D4:1 to D3:1, D4:2 to D3:2, D4:3 to D3:3, D1:6 to D3:4, D1:4 to D3:5, D5:1 to D4:1, D5:2 to D4:2, D5:3 to D4:3, D1:7 to D4:4, D1:8 to D4:5
Connections:
- net COL1: no longer SW10.2, SW14.2, SW18.2, SW21.2, SW22.2
- new net ROW4: SW10.2, SW14.2, SW18.2, SW21.2, SW22.2
Changed lines of the file:
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@@
 	)
 	(junction
-		(at 76.2 135.89)
-		(diameter 0)
-		(color 0 0 0 0)
-	)
-	(junction
 		(at 127 123.19)
 		(diameter 0)
@@
 	(wire
 		(pts
-			(xy 76.2 123.19) (xy 76.2 135.89)
+			(xy 76.2 123.19) (xy 76.2 148.59)
 		)
 		(stroke
@@
 	(wire
 		(pts
-			(xy 48.26 135.89) (xy 76.2 135.89)
+			(xy 48.26 135.89) (xy 96.52 135.89)
 		)
 		(stroke
@@
 	(wire
 		(pts
-			(xy 76.2 135.89) (xy 76.2 148.59)
-		)
-		(stroke
-			(width 0)
-			(type default)
-		)
-	)
-	(wire
-		(pts
 			(xy 152.4 97.79) (xy 157.48 97.79)
 		)
@@
 	(wire
 		(pts
-			(xy 76.2 135.89) (xy 96.52 135.89)
-		)
-		(stroke
-			(width 0)
-			(type default)
-		)
-	)
-	(wire
-		(pts
 			(xy 93.98 140.97) (xy 96.52 140.97)
 		)
@@
 		(dnp no)
 		(fields_autoplaced yes)
-		(property "Reference" "D4:1"
+		(property "Reference" "D3:1"
 			(at 83.82 116.84 0)
 			(effects
@@
 			(project "spur-demo"
 				(path "/48a1a14a-bba3-4ee0-af51-70720bbf1fda/e48efb72-302e-45b5-b9fb-6ddbb8e8c1ba"
-					(reference "D4:1")
+					(reference "D3:1")
 					(unit 1)
 				)
@@
 		(dnp no)
 		(fields_autoplaced yes)
-		(property "Reference" "D1:1"
+		(property "Reference" "D2:5"
 			(at 185.42 91.44 0)
 			(effects
@@
 			(project "spur-demo"
 				(path "/48a1a14a-bba3-4ee0-af51-70720bbf1fda/e48efb72-302e-45b5-b9fb-6ddbb8e8c1ba"
-					(reference "D1:1")
+					(reference "D2:5")
 					(unit 1)
 				)
@@
 		(dnp no)
 		(fields_autoplaced yes)
-		(property "Reference" "D3:1"
+		(property "Reference" "D2:1"
 			(at 83.82 91.44 0)
 			(effects
@@
 			(project "spur-demo"
 				(path "/48a1a14a-bba3-4ee0-af51-70720bbf1fda/e48efb72-302e-45b5-b9fb-6ddbb8e8c1ba"
-					(reference "D3:1")
+					(reference "D2:1")
 					(unit 1)
 				)
@@
 		(dnp no)
 		(fields_autoplaced yes)
-		(property "Reference" "D2:3"
+		(property "Reference" "D1:3"
 			(at 134.62 66.04 0)
 			(effects
@@
 			(project "spur-demo"
 				(path "/48a1a14a-bba3-4ee0-af51-70720bbf1fda/e48efb72-302e-45b5-b9fb-6ddbb8e8c1ba"
-					(reference "D2:3")
+					(reference "D1:3")
 					(unit 1)
 				)
@@
 		(dnp no)
 		(fields_autoplaced yes)
-		(property "Reference" "D1:2"
+		(property "Reference" "D1:4"
 			(at 160.02 66.04 0)
 			(effects
@@
 			(project "spur-demo"
 				(path "/48a1a14a-bba3-4ee0-af51-70720bbf1fda/e48efb72-302e-45b5-b9fb-6ddbb8e8c1ba"
-					(reference "D1:2")
+					(reference "D1:4")
 					(unit 1)
 				)
@@
 		(dnp no)
 		(fields_autoplaced yes)
-		(property "Reference" "D5:3"
+		(property "Reference" "D4:3"
 			(at 134.62 142.24 0)
 			(effects
@@
 			(project "spur-demo"
 				(path "/48a1a14a-bba3-4ee0-af51-70720bbf1fda/e48efb72-302e-45b5-b9fb-6ddbb8e8c1ba"
-					(reference "D5:3")
+					(reference "D4:3")
 					(unit 1)
 				)
@@
 		(dnp no)
 		(fields_autoplaced yes)
-		(property "Reference" "D2:1"
+		(property "Reference" "D1:1"
 			(at 83.82 66.04 0)
 			(effects
@@
 			(project "spur-demo"
 				(path "/48a1a14a-bba3-4ee0-af51-70720bbf1fda/e48efb72-302e-45b5-b9fb-6ddbb8e8c1ba"
-					(reference "D2:1")
+					(reference "D1:1")
 					(unit 1)
 				)
@@
 		(dnp no)
 		(fields_autoplaced yes)
-		(property "Reference" "D3:2"
+		(property "Reference" "D2:2"
 			(at 109.22 91.44 0)
 			(effects
@@
 			(project "spur-demo"
 				(path "/48a1a14a-bba3-4ee0-af51-70720bbf1fda/e48efb72-302e-45b5-b9fb-6ddbb8e8c1ba"
-					(reference "D3:2")
+					(reference "D2:2")
 					(unit 1)
 				)
@@
 		(dnp no)
 		(fields_autoplaced yes)
-		(property "Reference" "D1:3"
+		(property "Reference" "D2:4"
 			(at 160.02 91.44 0)
 			(effects
@@
 			(project "spur-demo"
 				(path "/48a1a14a-bba3-4ee0-af51-70720bbf1fda/e48efb72-302e-45b5-b9fb-6ddbb8e8c1ba"
-					(reference "D1:3")
+					(reference "D2:4")
 					(unit 1)
 				)
@@
 		(dnp no)
 		(fields_autoplaced yes)
-		(property "Reference" "D4:3"
+		(property "Reference" "D3:3"
 			(at 134.62 116.84 0)
 			(effects
@@
 			(project "spur-demo"
 				(path "/48a1a14a-bba3-4ee0-af51-70720bbf1fda/e48efb72-302e-45b5-b9fb-6ddbb8e8c1ba"
-					(reference "D4:3")
+					(reference "D3:3")
 					(unit 1)
 				)
@@
 		(dnp no)
 		(fields_autoplaced yes)
-		(property "Reference" "D3:3"
+		(property "Reference" "D2:3"
 			(at 134.62 91.44 0)
 			(effects
@@
 			(project "spur-demo"
 				(path "/48a1a14a-bba3-4ee0-af51-70720bbf1fda/e48efb72-302e-45b5-b9fb-6ddbb8e8c1ba"
-					(reference "D3:3")
+					(reference "D2:3")
 					(unit 1)
 				)
@@
 		(dnp no)
 		(fields_autoplaced yes)
-		(property "Reference" "D1:4"
+		(property "Reference" "D3:5"
 			(at 185.42 116.84 0)
 			(effects
@@
 			(project "spur-demo"
 				(path "/48a1a14a-bba3-4ee0-af51-70720bbf1fda/e48efb72-302e-45b5-b9fb-6ddbb8e8c1ba"
-					(reference "D1:4")
+					(reference "D3:5")
 					(unit 1)
 				)
@@
 		(dnp no)
 		(fields_autoplaced yes)
-		(property "Reference" "D1:8"
+		(property "Reference" "D4:5"
 			(at 185.42 142.24 0)
 			(effects
@@
 			(project "spur-demo"
 				(path "/48a1a14a-bba3-4ee0-af51-70720bbf1fda/e48efb72-302e-45b5-b9fb-6ddbb8e8c1ba"
-					(reference "D1:8")
+					(reference "D4:5")
 					(unit 1)
 				)
@@
 		(dnp no)
 		(fields_autoplaced yes)
-		(property "Reference" "D4:2"
+		(property "Reference" "D3:2"
 			(at 109.22 116.84 0)
 			(effects
@@
 			(project "spur-demo"
 				(path "/48a1a14a-bba3-4ee0-af51-70720bbf1fda/e48efb72-302e-45b5-b9fb-6ddbb8e8c1ba"
-					(reference "D4:2")
+					(reference "D3:2")
 					(unit 1)
 				)
@@
 		(dnp no)
 		(fields_autoplaced yes)
-		(property "Reference" "D1:7"
+		(property "Reference" "D4:4"
 			(at 160.02 142.24 0)
 			(effects
@@
 			(project "spur-demo"
 				(path "/48a1a14a-bba3-4ee0-af51-70720bbf1fda/e48efb72-302e-45b5-b9fb-6ddbb8e8c1ba"
-					(reference "D1:7")
+					(reference "D4:4")
 					(unit 1)
 				)
@@
 		(dnp no)
 		(fields_autoplaced yes)
-		(property "Reference" "D1:6"
+		(property "Reference" "D3:4"
 			(at 160.02 116.84 0)
 			(effects
@@
 			(project "spur-demo"
 				(path "/48a1a14a-bba3-4ee0-af51-70720bbf1fda/e48efb72-302e-45b5-b9fb-6ddbb8e8c1ba"
-					(reference "D1:6")
+					(reference "D3:4")
 					(unit 1)
 				)
@@
 		(dnp no)
 		(fields_autoplaced yes)
-		(property "Reference" "D2:2"
+		(property "Reference" "D1:2"
 			(at 109.22 66.04 0)
 			(effects
@@
 			(project "spur-demo"
 				(path "/48a1a14a-bba3-4ee0-af51-70720bbf1fda/e48efb72-302e-45b5-b9fb-6ddbb8e8c1ba"
-					(reference "D2:2")
+					(reference "D1:2")
 					(unit 1)
 				)
@@
 		(dnp no)
 		(fields_autoplaced yes)
-		(property "Reference" "D5:1"
+		(property "Reference" "D4:1"
 			(at 83.82 142.24 0)
 			(effects
@@
 			(project "spur-demo"
 				(path "/48a1a14a-bba3-4ee0-af51-70720bbf1fda/e48efb72-302e-45b5-b9fb-6ddbb8e8c1ba"
-					(reference "D5:1")
+					(reference "D4:1")
 					(unit 1)
 				)
@@
 		(dnp no)
 		(fields_autoplaced yes)
-		(property "Reference" "D5:2"
+		(property "Reference" "D4:2"
 			(at 109.22 142.24 0)
 			(effects
@@
 			(project "spur-demo"
 				(path "/48a1a14a-bba3-4ee0-af51-70720bbf1fda/e48efb72-302e-45b5-b9fb-6ddbb8e8c1ba"
-					(reference "D5:2")
+					(reference "D4:2")
 					(unit 1)
 				)

Commit message: docs: add application note for keypad scanning
Other:
- note added: "Keypad Matrix Application Note: The ROW pins get pulled up by the GPIO expander, with one ROW being pulled down. The scanner relies on the COL pins being read in as a logic swing to low. Remarked as Domino Logic, a rail-to-rail logic swing occurs."
- moved on the sheet: D1:1, D1:2, D1:3, D1:4, D1:5, D2:1, D2:2, D2:3, D2:4, D2:5, D3:1, D3:2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

Commit message: fix: geographically reannotate keypad DTMF matrix
Parts:
- renumbered SW5 to SW10, SW15 to SW11, SW16 to SW12, SW17 to SW13, SW20 to SW14, SW10 to SW15, SW14 to SW16, SW18 to SW17, SW21 to SW18, SW3 to SW20, SW6 to SW21, SW7 to SW3, SW8 to SW4, SW9 to SW5, SW4 to SW6, SW11 to SW7, SW12 to SW8, SW13 to SW9
Changed lines of the file:
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@@
 		(on_board yes)
 		(dnp no)
-		(property "Reference" "SW8"
+		(property "Reference" "SW4"
 			(at 79.756 53.34 90)
 			(effects
@@
 			(project "spur-demo"
 				(path "/48a1a14a-bba3-4ee0-af51-70720bbf1fda/e48efb72-302e-45b5-b9fb-6ddbb8e8c1ba"
-					(reference "SW8")
+					(reference "SW4")
 					(unit 1)
 				)
@@
 		(on_board yes)
 		(dnp no)
-		(property "Reference" "SW17"
+		(property "Reference" "SW13"
 			(at 105.156 104.14 90)
 			(effects
@@
 			(project "spur-demo"
 				(path "/48a1a14a-bba3-4ee0-af51-70720bbf1fda/e48efb72-302e-45b5-b9fb-6ddbb8e8c1ba"
-					(reference "SW17")
+					(reference "SW13")
 					(unit 1)
 				)
@@
 		(on_board yes)
 		(dnp no)
-		(property "Reference" "SW7"
+		(property "Reference" "SW3"
 			(at 54.356 53.34 90)
 			(effects
@@
 			(project "spur-demo"
 				(path "/48a1a14a-bba3-4ee0-af51-70720bbf1fda/e48efb72-302e-45b5-b9fb-6ddbb8e8c1ba"
-					(reference "SW7")
+					(reference "SW3")
 					(unit 1)
 				)
@@
 		(on_board yes)
 		(dnp no)
-		(property "Reference" "SW15"
+		(property "Reference" "SW11"
 			(at 54.356 104.14 90)
 			(effects
@@
 			(project "spur-demo"
 				(path "/48a1a14a-bba3-4ee0-af51-70720bbf1fda/e48efb72-302e-45b5-b9fb-6ddbb8e8c1ba"
-					(reference "SW15")
+					(reference "SW11")
 					(unit 1)
 				)
@@
 		(on_board yes)
 		(dnp no)
-		(property "Reference" "SW9"
+		(property "Reference" "SW5"
 			(at 105.156 53.34 90)
 			(effects
@@
 			(project "spur-demo"
 				(path "/48a1a14a-bba3-4ee0-af51-70720bbf1fda/e48efb72-302e-45b5-b9fb-6ddbb8e8c1ba"
-					(reference "SW9")
+					(reference "SW5")
 					(unit 1)
 				)
@@
 		(on_board yes)
 		(dnp no)
-		(property "Reference" "SW16"
+		(property "Reference" "SW12"
 			(at 79.756 104.14 90)
 			(effects
@@
 			(project "spur-demo"
 				(path "/48a1a14a-bba3-4ee0-af51-70720bbf1fda/e48efb72-302e-45b5-b9fb-6ddbb8e8c1ba"
-					(reference "SW16")
+					(reference "SW12")
 					(unit 1)
 				)
@@
 		(on_board yes)
 		(dnp no)
-		(property "Reference" "SW10"
+		(property "Reference" "SW15"
 			(at 54.356 129.54 90)
 			(effects
@@
 			(project "spur-demo"
 				(path "/48a1a14a-bba3-4ee0-af51-70720bbf1fda/e48efb72-302e-45b5-b9fb-6ddbb8e8c1ba"
-					(reference "SW10")
+					(reference "SW15")
 					(unit 1)
 				)
@@
 		(on_board yes)
 		(dnp no)
-		(property "Reference" "SW11"
+		(property "Reference" "SW7"
 			(at 54.356 78.74 90)
 			(effects
@@
 			(project "spur-demo"
 				(path "/48a1a14a-bba3-4ee0-af51-70720bbf1fda/e48efb72-302e-45b5-b9fb-6ddbb8e8c1ba"
-					(reference "SW11")
+					(reference "SW7")
 					(unit 1)
 				)
@@
 		(on_board yes)
 		(dnp no)
-		(property "Reference" "SW21"
+		(property "Reference" "SW18"
 			(at 130.556 129.54 90)
 			(effects
@@
 			(project "spur-demo"
 				(path "/48a1a14a-bba3-4ee0-af51-70720bbf1fda/e48efb72-302e-45b5-b9fb-6ddbb8e8c1ba"
-					(reference "SW21")
+					(reference "SW18")
 					(unit 1)
 				)
@@
 		(on_board yes)
 		(dnp no)
-		(property "Reference" "SW20"
+		(property "Reference" "SW14"
 			(at 130.556 104.14 90)
 			(effects
@@
 			(project "spur-demo"
 				(path "/48a1a14a-bba3-4ee0-af51-70720bbf1fda/e48efb72-302e-45b5-b9fb-6ddbb8e8c1ba"
-					(reference "SW20")
+					(reference "SW14")
 					(unit 1)
 				)
@@
 		(on_board yes)
 		(dnp no)
-		(property "Reference" "SW3"
+		(property "Reference" "SW20"
 			(at 155.956 78.74 90)
 			(effects
@@
 			(project "spur-demo"
 				(path "/48a1a14a-bba3-4ee0-af51-70720bbf1fda/e48efb72-302e-45b5-b9fb-6ddbb8e8c1ba"
-					(reference "SW3")
+					(reference "SW20")
 					(unit 1)
 				)
@@
 		(on_board yes)
 		(dnp no)
-		(property "Reference" "SW12"
+		(property "Reference" "SW8"
 			(at 79.756 78.74 90)
 			(effects
@@
 			(project "spur-demo"
 				(path "/48a1a14a-bba3-4ee0-af51-70720bbf1fda/e48efb72-302e-45b5-b9fb-6ddbb8e8c1ba"
-					(reference "SW12")
+					(reference "SW8")
 					(unit 1)
 				)
@@
 		(on_board yes)
 		(dnp no)
-		(property "Reference" "SW4"
+		(property "Reference" "SW6"
 			(at 130.556 53.34 90)
 			(effects
@@
 			(project "spur-demo"
 				(path "/48a1a14a-bba3-4ee0-af51-70720bbf1fda/e48efb72-302e-45b5-b9fb-6ddbb8e8c1ba"
-					(reference "SW4")
+					(reference "SW6")
 					(unit 1)
 				)
@@
 		(on_board yes)
 		(dnp no)
-		(property "Reference" "SW6"
+		(property "Reference" "SW21"
 			(at 155.956 104.14 90)
 			(effects
@@
 			(project "spur-demo"
 				(path "/48a1a14a-bba3-4ee0-af51-70720bbf1fda/e48efb72-302e-45b5-b9fb-6ddbb8e8c1ba"
-					(reference "SW6")
+					(reference "SW21")
 					(unit 1)
 				)
@@
 		(on_board yes)
 		(dnp no)
-		(property "Reference" "SW18"
+		(property "Reference" "SW17"
 			(at 105.156 129.54 90)
 			(effects
@@
 			(project "spur-demo"
 				(path "/48a1a14a-bba3-4ee0-af51-70720bbf1fda/e48efb72-302e-45b5-b9fb-6ddbb8e8c1ba"
-					(reference "SW18")
+					(reference "SW17")
 					(unit 1)
 				)
@@
 		(on_board yes)
 		(dnp no)
-		(property "Reference" "SW14"
+		(property "Reference" "SW16"
 			(at 79.756 129.54 90)
 			(effects
@@
 			(project "spur-demo"
 				(path "/48a1a14a-bba3-4ee0-af51-70720bbf1fda/e48efb72-302e-45b5-b9fb-6ddbb8e8c1ba"
-					(reference "SW14")
+					(reference "SW16")
 					(unit 1)
 				)
@@
 		(on_board yes)
 		(dnp no)
-		(property "Reference" "SW5"
+		(property "Reference" "SW10"
 			(at 130.556 78.74 90)
 			(effects
@@
 			(project "spur-demo"
 				(path "/48a1a14a-bba3-4ee0-af51-70720bbf1fda/e48efb72-302e-45b5-b9fb-6ddbb8e8c1ba"
-					(reference "SW5")
+					(reference "SW10")
 					(unit 1)
 				)
@@
 		(on_board yes)
 		(dnp no)
-		(property "Reference" "SW13"
+		(property "Reference" "SW9"
 			(at 105.156 78.74 90)
 			(effects
@@
 			(project "spur-demo"
 				(path "/48a1a14a-bba3-4ee0-af51-70720bbf1fda/e48efb72-302e-45b5-b9fb-6ddbb8e8c1ba"
-					(reference "SW13")
+					(reference "SW9")
 					(unit 1)
 				)

Commit message: feat: squash recaptured schematics and footprint reassignments
Parts:
- added H1, H2: MountingHole_2.2mm_M2_Pad_Via, MountingHole:MountingHole_2.2mm_M2_Pad_Via, symbol Mechanical:MountingHole
- added J6: Conn_01x08_Socket, spur-demo:HW-834, symbol Connector:Conn_01x08_Socket
- D1:1, D1:2, D1:3, D1:4, D1:5, D2:1, D2:2, D2:3, D2:4, D2:5, D3:1, D3:2, D3:3, D3:4, D3:5, D4:1, D4:2, D4:3, D4:4, D4:5, SW10, SW11, SW12, SW13, SW14, SW15, SW16, SW17, SW18, SW19, SW20, SW21, SW22, SW3, SW4, SW5, SW6, SW7, SW8, SW9: now not fitted; now left out of the parts list
Connections:
- net COL1: now also J6.5 (Pin_5)
- net COL2: now also J6.6 (Pin_6)
- net COL3: now also J6.7 (Pin_7)
- net COL4: now also J6.8 (Pin_8)
- net ROW1: now also J6.4 (Pin_4)
- net ROW2: now also J6.3 (Pin_3)
- net ROW3: now also J6.2 (Pin_2)
- net ROW4: now also J6.1 (Pin_1)
