File: Hardware/KiCAD/spur-demo/keypad.kicad_sch (KiCad schematic)
At the start: 43 parts, among them J6 Conn_01x08_Socket, SW10 DOWN, SW11 7, SW12 8, SW13 9, SW14 LEFT, SW15 *, SW16 0, SW17 #, SW18 RIGHT, SW19 PTT, SW20 MENU, SW21 EXIT, SW22 SK0, SW3 1, SW4 2, SW5 3, SW6 UP, SW7 4, SW8 5, SW9 6

Commit message: fix: select correct standoff size in schematic
Parts:
- H1, H2: value MountingHole_2.2mm_M2_Pad_Via -> MountingHole_2.7mm_M2_Pad_Via; footprint MountingHole:MountingHole_2.2mm_M2_Pad_Via -> MountingHole:MountingHole_2.7mm_Pad_Via
Other:
- moved on the sheet: H2
Changed lines of the file:
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@@
 	(symbol
 		(lib_id "Mechanical:MountingHole")
-		(at 220.98 105.41 0)
+		(at 203.2 111.76 0)
 		(unit 1)
 		(exclude_from_sim yes)
@@
 		(fields_autoplaced yes)
 		(property "Reference" "H2"
-			(at 223.52 104.1399 0)
+			(at 205.74 110.4899 0)
 			(effects
 				(font
@@
 			)
 		)
-		(property "Value" "MountingHole_2.2mm_M2_Pad_Via"
-			(at 223.52 106.6799 0)
+		(property "Value" "MountingHole_2.7mm_M2_Pad_Via"
+			(at 205.74 113.0299 0)
 			(effects
 				(font
@@
 			)
 		)
-		(property "Footprint" "MountingHole:MountingHole_2.2mm_M2_Pad_Via"
-			(at 220.98 105.41 0)
-			(effects
-				(font
-					(size 1.27 1.27)
-				)
-				(hide yes)
-			)
-		)
-		(property "Datasheet" "~"
-			(at 220.98 105.41 0)
+		(property "Footprint" "MountingHole:MountingHole_2.7mm_Pad_Via"
+			(at 203.2 111.76 0)
+			(effects
+				(font
+					(size 1.27 1.27)
+				)
+				(hide yes)
+			)
+		)
+		(property "Datasheet" "~"
+			(at 203.2 111.76 0)
 			(effects
 				(font
@@
 		)
 		(property "Description" ""
-			(at 220.98 105.41 0)
+			(at 203.2 111.76 0)
 			(effects
 				(font
@@
 			)
 		)
-		(property "Value" "MountingHole_2.2mm_M2_Pad_Via"
+		(property "Value" "MountingHole_2.7mm_M2_Pad_Via"
 			(at 205.74 106.6799 0)
 			(effects
@@
 			)
 		)
-		(property "Footprint" "MountingHole:MountingHole_2.2mm_M2_Pad_Via"
+		(property "Footprint" "MountingHole:MountingHole_2.7mm_Pad_Via"
 			(at 203.2 105.41 0)
 			(effects
