File: Hardware/KiCAD/spur-demo/power_subsystem.kicad_sch (KiCad schematic)
At the start: 29 parts, among them IC1 BQ24193RGER, IC3 ISL91127IRNZ-T7A, J5 Screw_Terminal_01x02, Q1 IRLZ44N

Commit message: feat: add stat & pg indicators, psel solder jumper, begin power switch
Parts:
- added D5, D6: LED, symbol Device:LED
- added JP7: PSEL, symbol Jumper:SolderJumper_3_Bridged12
- added R38, R39: 2.2k, symbol Device:R_US
Connections:
- net 3.3V: now also JP7.1 (A); no longer IC1.2 (PSEL)
- net GND: now also JP7.3 (B)
- net V_{SYS}: now also D5.2 (A), D6.2 (A)
- net ~{PG}: now reaches IC1.3 (~{PG})
- net ~{PG}: now also R39.2
- net STAT: now reaches IC1.4 (STAT)
- net STAT: now also R38.2
- new net: D6.1 (K), R39.1
- new net: D5.1 (K), R38.1
- new net: IC1.2 (PSEL), JP7.2 (C)
- no-connect marks 2 -> 0
Other:
- moved on the sheet: C1, C10, C11, C12, C2, C3, C4, C5, C6, C7, C8, C9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

Commit message: feat: begin footprint assignment, unify +3.3V PWRREFs
Parts:
- D5, D6: footprint (none) -> LED_SMD:LED_0603_1608Metric_Pad1.05x0.95mm_HandSolder
- R38, R39: footprint (none) -> Resistor_SMD:R_0603_1608Metric
- TH1: footprint bms-smps-testbench:103AT2 -> spur-demo:103AT2
Connections:
- net 3.3V renamed +3.3V
Changed lines of the file:
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@@
 			)
 		)
-		(property "Footprint" ""
+		(property "Footprint" "Resistor_SMD:R_0603_1608Metric"
 			(at 114.554 38.354 90)
 			(effects
@@
 			)
 		)
-		(property "Value" "3.3V"
+		(property "Value" "+3.3V"
 			(at 243.84 29.21 0)
 			(effects
@@
 			)
 		)
-		(property "Footprint" ""
+		(property "Footprint" "Resistor_SMD:R_0603_1608Metric"
 			(at 114.554 28.194 90)
 			(effects
@@
 			)
 		)
-		(property "Footprint" ""
+		(property "Footprint" "LED_SMD:LED_0603_1608Metric_Pad1.05x0.95mm_HandSolder"
 			(at 104.14 39.37 0)
 			(effects
@@
 			)
 		)
-		(property "Footprint" "bms-smps-testbench:103AT2"
+		(property "Footprint" "spur-demo:103AT2"
 			(at 104.14 59.69 0)
 			(effects
@@
 			)
 		)
-		(property "Value" "3.3V"
+		(property "Value" "+3.3V"
 			(at 22.86 62.23 0)
 			(effects
@@
 			)
 		)
-		(property "Footprint" ""
+		(property "Footprint" "LED_SMD:LED_0603_1608Metric_Pad1.05x0.95mm_HandSolder"
 			(at 104.14 29.21 0)
 			(effects
@@
 			)
 		)
-		(property "Value" "3.3V"
+		(property "Value" "+3.3V"
 			(at 34.29 19.05 0)
 			(effects

Commit message: feat: assign solder jumper footprints, begin testpoints
Parts:
- JP7: footprint (none) -> Jumper:SolderJumper-3_P1.3mm_Bridged12_RoundedPad1.0x1.5mm_NumberLabels
Changed lines of the file:
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@@
 			)
 		)
-		(property "Footprint" ""
+		(property "Footprint" "Jumper:SolderJumper-3_P1.3mm_Bridged12_RoundedPad1.0x1.5mm_NumberLabels"
 			(at 22.86 74.93 0)
 			(effects

Commit message: feat: phase out screw terminals in favor of real connectors
Parts:
- J5: value Screw_Terminal_01x02 -> Conn_01x02; footprint TerminalBlock_Phoenix:TerminalBlock_Phoenix_MPT-0,5-2-2.54_1x02_P2.54mm_Horizontal -> Connector_JST:JST_GH_SM02B-GHS-TB_1x02-1MP_P1.25mm_Horizontal; symbol Connector:Screw_Terminal_01x02 -> Connector_Generic:Conn_01x02
Changed lines of the file:
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@@
 	)
 	(symbol
-		(lib_id "Connector:Screw_Terminal_01x02")
+		(lib_id "Connector_Generic:Conn_01x02")
 		(at 115.57 111.76 0)
 		(unit 1)
@@
 			)
 		)
-		(property "Value" "Screw_Terminal_01x02"
+		(property "Value" "Conn_01x02"
 			(at 118.11 114.2999 0)
 			(effects
@@
 			)
 		)
-		(property "Footprint" "TerminalBlock_Phoenix:TerminalBlock_Phoenix_MPT-0,5-2-2.54_1x02_P2.54mm_Horizontal"
+		(property "Footprint" "Connector_JST:JST_GH_SM02B-GHS-TB_1x02-1MP_P1.25mm_Horizontal"
 			(at 115.57 111.76 0)
 			(effects
@@
 			)
 		)
-		(property "Description" "Generic screw terminal, single row, 01x02, script generated (kicad-library-utils/schlib/autogen/connector/)"
+		(property "Description" "Generic connector, single row, 01x02, script generated (kicad-library-utils/schlib/autogen/connector/)"
 			(at 115.57 111.76 0)
 			(effects

Commit message: feat: squash recaptured schematics and footprint reassignments
Parts:
- added BT2: 1122, spur-demo:BAT_1122, symbol spur-demo:1122
- J5: now not fitted
- Q1: value IRLZ44N -> ZXMN2A01F; footprint Package_TO_SOT_THT:TO-220-3_Vertical -> Package_TO_SOT_SMD:SOT-23; symbol Transistor_FET:IRLZ44N -> Transistor_FET:ZXMN2A01F
Connections:
- net +3.3V: no longer JP7.1 (A), R1.1
- net +BATT: now also BT2.P
- net GND: now also BT2.N
- net at C8.2, C9.2, IC3.10 (VIN)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: now also Q1.2 (S); no longer Q1.3 (S)
- net V_{SYS} renamed +SYS
- net +SYS: now also JP7.1 (A), Q1.3 (D), R1.1; no longer Q1.2 (D)
Other:
- moved on the sheet: C7, D5, D6, R38, R39
