File: Hardware/KiCAD/spur-demo/power_subsystem.kicad_sch (KiCad schematic)
At the start: 35 parts, among them IC1 BQ24193RGER, IC3 ISL91127IRNZ-T7A, J5 Conn_01x02, Q1 ZXMN2A01F

Commit message: feat: completely reroute demo PCB, zones still not fully connected
Parts:
- J5: footprint Connector_JST:JST_GH_SM02B-GHS-TB_1x02-1MP_P1.25mm_Horizontal -> Connector_PinHeader_2.54mm:PinHeader_1x02_P2.54mm_Vertical; now fitted
Changed lines of the file:
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@@
 		(in_bom yes)
 		(on_board yes)
-		(dnp yes)
+		(dnp no)
 		(fields_autoplaced yes)
 		(property "Reference" "J5"
@@
 			)
 		)
-		(property "Footprint" "Connector_JST:JST_GH_SM02B-GHS-TB_1x02-1MP_P1.25mm_Horizontal"
+		(property "Footprint" "Connector_PinHeader_2.54mm:PinHeader_1x02_P2.54mm_Vertical"
 			(at 115.57 111.76 0)
 			(effects

Commit message: fix: correct NTC thermistor resistor network
Connections:
- net TS_P is gone; now on an unnamed net: IC1.11 (TS1), IC1.12 (TS2), TH1.2
- net GND: now also TH1.1
- net TS_N: no longer names the net of R2.1, R3.2
- net TS_N: no longer TH1.1
Other:
- moved on the sheet: R2, R3, TH1
