File: Hardware/KiCAD/spur-demo/spur-demo.kicad_sch (KiCad schematic)
At the start: 12 parts, among them IC2 PCF8575PWR, J1 Peripherals, J12 USB_C_Plug_USB2.0, J2 Conn_Coaxial, U1 SA868

Commit message: feat: begin footprint assignment, unify +3.3V PWRREFs
Parts:
- C18: footprint Capacitor_SMD:C_0603_1608Metric -> Capacitor_SMD:C_0603_1608Metric_Pad1.08x0.95mm_HandSolder
- D1: footprint SP0503BAHTG:SOT143 -> Package_TO_SOT_SMD:SOT-143_Handsoldering; symbol Cobalt-Cowboy:SP0503BAHTG -> spur-demo:SP0503BAHTG
- IC2: footprint Cobalt_Cowboy:SOP65P640X120-24N_PCF8575PWR -> spur-demo:SOP65P640X120-24N_PCF8575PWR; symbol Cobalt-Cowboy:PCF8575PWR -> spur-demo:PCF8575PWR
Connections:
- net 3.3V is gone; now on net +3.3V: IC2.24 (VCC), J1.1 (Pin_1)
- net BMS_OTG: now also IC2.6 (P02); no longer IC2.5 (P01)
- net ~{AMP_SD}: now also IC2.7 (P03); no longer IC2.6 (P02)
- net ~{RADIO_PD}: now also IC2.8 (P04); no longer IC2.7 (P03)
- net ~{RADIO_PTT}: now also IC2.9 (P05); no longer IC2.8 (P04)
- net ~{SPIM2_CS}: now also IC2.10 (P06); no longer IC2.9 (P05)
- new net ~{BMS_PG}: IC2.5 (P01)
- no-connect marks 30 -> 29
Other:
- sheet Power Subsystem ports: added ~{PG}; removed none
Changed lines of the file:
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@@
 	)
 	(no_connect
-		(at 55.88 166.37)
-	)
-	(no_connect
 		(at 167.64 176.53)
 	)
@@
 	(wire
 		(pts
-			(xy 57.15 88.9) (xy 57.15 91.44)
-		)
-		(stroke
-			(width 0)
-			(type default)
-		)
-	)
-	(wire
-		(pts
 			(xy 124.46 69.85) (xy 137.16 69.85)
 		)
@@
 	(wire
 		(pts
-			(xy 46.99 163.83) (xy 58.42 163.83)
+			(xy 46.99 166.37) (xy 58.42 166.37)
 		)
 		(stroke
@@
 	(wire
 		(pts
+			(xy 57.15 88.9) (xy 57.15 91.44)
+		)
+		(stroke
+			(width 0)
+			(type default)
+		)
+	)
+	(wire
+		(pts
 			(xy 86.36 161.29) (xy 99.06 161.29)
 		)
@@
 	(wire
 		(pts
+			(xy 58.42 153.67) (xy 46.99 153.67)
+		)
+		(stroke
+			(width 0)
+			(type default)
+		)
+	)
+	(wire
+		(pts
 			(xy 86.36 156.21) (xy 99.06 156.21)
 		)
@@
 	(wire
 		(pts
-			(xy 46.99 161.29) (xy 58.42 161.29)
+			(xy 46.99 163.83) (xy 58.42 163.83)
 		)
 		(stroke
@@
 	(wire
 		(pts
-			(xy 46.99 156.21) (xy 58.42 156.21)
+			(xy 46.99 158.75) (xy 58.42 158.75)
 		)
 		(stroke
@@
 	(wire
 		(pts
-			(xy 55.88 166.37) (xy 58.42 166.37)
+			(xy 209.55 57.15) (xy 195.58 57.15)
 		)
 		(stroke
@@
 	(wire
 		(pts
-			(xy 209.55 57.15) (xy 195.58 57.15)
+			(xy 229.87 41.91) (xy 240.03 41.91)
 		)
 		(stroke
@@
 	(wire
 		(pts
-			(xy 58.42 153.67) (xy 46.99 153.67)
+			(xy 58.42 156.21) (xy 46.99 156.21)
 		)
 		(stroke
@@
 	(wire
 		(pts
-			(xy 58.42 158.75) (xy 46.99 158.75)
+			(xy 58.42 161.29) (xy 46.99 161.29)
 		)
 		(stroke
@@
 		)
 	)
+	(label "~{BMS_PG}"
+		(at 46.99 153.67 0)
+		(fields_autoplaced yes)
+		(effects
+			(font
+				(size 1.27 1.27)
+			)
+			(justify left bottom)
+		)
+	)
 	(label "A2"
 		(at 26.67 177.8 0)
@@
 		)
 	)
+	(label "~{BMS_PG}"
+		(at 240.03 41.91 180)
+		(fields_autoplaced yes)
+		(effects
+			(font
+				(size 1.27 1.27)
+			)
+			(justify right bottom)
+		)
+	)
 	(label "~{SPIM2_CS}"
 		(at 121.92 163.83 0)
@@
 	)
 	(label "~{RADIO_PD}"
-		(at 46.99 158.75 0)
+		(at 46.99 161.29 0)
 		(fields_autoplaced yes)
 		(effects
@@
 	)
 	(label "~{SPIM2_CS}"
-		(at 46.99 163.83 0)
+		(at 46.99 166.37 0)
 		(fields_autoplaced yes)
 		(effects
@@
 	)
 	(label "~{RADIO_PTT}"
-		(at 46.99 161.29 0)
+		(at 46.99 163.83 0)
 		(fields_autoplaced yes)
 		(effects
@@
 	)
 	(label "BMS_OTG"
-		(at 46.99 153.67 0)
+		(at 46.99 156.21 0)
 		(fields_autoplaced yes)
 		(effects
@@
 	)
 	(label "~{AMP_SD}"
-		(at 46.99 156.21 0)
+		(at 46.99 158.75 0)
 		(fields_autoplaced yes)
 		(effects
@@
 			)
 		)
-		(property "Footprint" "Capacitor_SMD:C_0603_1608Metric"
+		(property "Footprint" "Capacitor_SMD:C_0603_1608Metric_Pad1.08x0.95mm_HandSolder"
 			(at 100.0252 39.37 0)
 			(effects
@@
 	)
 	(symbol
-		(lib_id "Cobalt-Cowboy:PCF8575PWR")
+		(lib_id "spur-demo:PCF8575PWR")
 		(at 58.42 143.51 0)
 		(unit 1)
@@
 			)
 		)
-		(property "Footprint" "Cobalt_Cowboy:SOP65P640X120-24N_PCF8575PWR"
+		(property "Footprint" "spur-demo:SOP65P640X120-24N_PCF8575PWR"
 			(at 82.55 238.43 0)
 			(effects
@@
 	)
 	(symbol
-		(lib_id "Cobalt-Cowboy:SP0503BAHTG")
+		(lib_id "spur-demo:SP0503BAHTG")
 		(at 67.31 62.23 270)
 		(mirror x)
@@
 			)
 		)
-		(property "Footprint" "SP0503BAHTG:SOT143"
+		(property "Footprint" "Package_TO_SOT_SMD:SOT-143_Handsoldering"
 			(at 67.31 62.23 0)
 			(effects
@@
 			)
 		)
-		(property "Value" "3.3V"
+		(property "Value" "+3.3V"
 			(at 88.9 135.89 0)
 			(effects
@@
 			)
 		)
-		(property "Value" "3.3V"
+		(property "Value" "+3.3V"
 			(at 27.94 146.05 0)
 			(effects
@@
 			)
 		)
+		(pin "~{PG}" output
+			(at 229.87 41.91 0)
+			(effects
+				(font
+					(size 1.27 1.27)
+				)
+				(justify right)
+			)
+		)

Commit message: feat: use smaller 1N5819 diode footprint 0603 imperial
Parts:
- D2: footprint Diode_THT:D_DO-41_SOD81_P10.16mm_Horizontal -> Diode_SMD:D_0603_1608Metric_Pad1.05x0.95mm_HandSolder
Changed lines of the file:
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@@
 			)
 		)
-		(property "Footprint" "Diode_THT:D_DO-41_SOD81_P10.16mm_Horizontal"
+		(property "Footprint" "Diode_SMD:D_0603_1608Metric_Pad1.05x0.95mm_HandSolder"
 			(at 92.71 33.655 0)
 			(effects

Commit message: feat: add solder jumper for usb current limit select
Parts:
- added JP11: OTG, Jumper:SolderJumper-3_P1.3mm_Bridged12_RoundedPad1.0x1.5mm_NumberLabels, symbol Jumper:SolderJumper_3_Bridged12
Connections:
- net +3.3V: now also JP11.1 (A)
- net BMS_OTG: now also JP11.2 (C); no longer IC2.6 (P02)
- net GND: now also JP11.3 (B)
- net ~{AMP_SD}: now also IC2.8 (P04); no longer IC2.7 (P03)
- net ~{RADIO_PD}: now also IC2.9 (P05); no longer IC2.8 (P04)
- net ~{RADIO_PTT}: now also IC2.10 (P06); no longer IC2.9 (P05)
- net ~{SPIM2_CS}: now also IC2.6 (P02); no longer IC2.10 (P06)
- new net OLED_D/~{C}: IC2.7 (P03)
- no-connect marks 29 -> 28

Commit message: feat: squash recaptured schematics and footprint reassignments
Parts:
- removed J1: Peripherals, Connector_JST:JST_EH_B4B-EH-A_1x04_P2.50mm_Vertical, symbol Connector_Generic:Conn_01x04
- added J1: SSD1306 Module, spur-demo:SSD1306, symbol Connector:Conn_01x04_Socket
- R26: value 5.1K -> 56k
- R27: value 5.1k -> 56k
Connections:
- net +3.3V: now also J1.1 (Pin_1); no longer JP11.1 (A)
- net GND: now also J1.2 (Pin_2)
- net I2C0_SCL: now also J1.3 (Pin_3)
- net I2C0_SDA: now also J1.4 (Pin_4)
- net ~{BMS_PG}: no longer names the net of IC2.5 (P01)
- new net +SYS: JP11.1 (A)
- no-connect marks 28 -> 34
Other:
- sheet Computing Subsystem ports: added ~{SD_CS}; removed none
- sheet Power Subsystem ports: added none; removed ~{PG}
- note added: "Configuration Channel R_{A5}, R_{B5} USB DFP Legacy Mode"
- note added: "Display Module over SPIM2 @ ~{SPIM2_CS}=0 In prototype, display module is I2C @0x3D"
- note removed: "Display Module over SPIM2 @ ~{SPIM2_CS}=0"
