File: Hardware/KiCAD/spur-demo/spur-demo.kicad_sch (KiCad schematic)
At the start: 13 parts, among them IC2 PCF8575PWR, J1 SSD1306 Module, J12 USB_C_Plug_USB2.0, J2 Conn_Coaxial, U1 SA868

Commit message: feat: add rotary encoder to demo board
Parts:
- added SW23: RotaryEncoder_Switch, RotaryEncoder_Bourns_Horizontal_PEC12R-2x17F-Sxxxx, symbol Device:RotaryEncoder_Switch
Connections:
- net OLED_D/~{C} is gone; now on net ~{BMS_CE}: IC2.7 (P03)
- net +3.3V: now also SW23.C
- net GND: now also SW23.S2
- net ~{BMS_CE}: no longer IC2.4 (P00)
- net ENC_DT: now reaches IC2.5 (P01)
- net ENC_DT: now also SW23.B
- new net ENC_CLK: IC2.4 (P00), SW23.A
- new net ENC_SW: SW23.S1
- no-connect marks 34 -> 33

Commit message: chore: specify encoder footprint, replot demo schematic
Parts:
- SW23: footprint RotaryEncoder_Bourns_Horizontal_PEC12R-2x17F-Sxxxx -> Rotary_Encoder:RotaryEncoder_Bourns_Horizontal_PEC12R-2x17F-Sxxxx
Changed lines of the file:
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@@
 			)
 		)
-		(property "Footprint" "RotaryEncoder_Bourns_Horizontal_PEC12R-2x17F-Sxxxx"
+		(property "Footprint" "Rotary_Encoder:RotaryEncoder_Bourns_Horizontal_PEC12R-2x17F-Sxxxx"
 			(at 201.93 147.066 0)
 			(effects

Commit message: chore: clarify confused use of PORT07 in prototype firmware and COL5 for switch matrix
Connections:
- net Keypad/COL5 is gone; now on net ENC_SW: IC2.11 (P07)
Other:
- note added: "TODO: reconcile use of PORT07 as ENC_SW and COL5"
Changed lines of the file:
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@@
 		)
 	)
+	(text "TODO: reconcile use of PORT07\nas ENC_SW and COL5"
+		(exclude_from_sim no)
+		(at 15.24 147.32 0)
+		(effects
+			(font
+				(size 1.27 1.27)
+			)
+			(justify left)
+		)
+	)
 	(text "I2C BUS ADDRESSING\nREAD = 0x41\nWRITE = 0x40"
 		(exclude_from_sim no)
-		(at 26.162 188.214 0)
+		(at 18.542 188.214 0)
 		(effects
 			(font
@@
 	)
 	(junction
+		(at 53.34 176.53)
+		(diameter 0)
+		(color 0 0 0 0)
+	)
+	(junction
 		(at 39.37 115.57)
 		(diameter 0)
@@
 	(wire
 		(pts
-			(xy 43.18 172.72) (xy 26.67 172.72)
+			(xy 35.56 172.72) (xy 19.05 172.72)
 		)
 		(stroke
@@
 	(wire
 		(pts
-			(xy 33.02 177.8) (xy 33.02 180.34)
+			(xy 25.4 177.8) (xy 25.4 180.34)
 		)
 		(stroke
@@
 	(wire
 		(pts
-			(xy 38.1 175.26) (xy 26.67 175.26)
+			(xy 30.48 175.26) (xy 19.05 175.26)
 		)
 		(stroke
@@
 	(wire
 		(pts
+			(xy 44.45 176.53) (xy 53.34 176.53)
+		)
+		(stroke
+			(width 0)
+			(type default)
+		)
+	)
+	(wire
+		(pts
 			(xy 182.88 54.61) (xy 171.45 54.61)
 		)
@@
 	(wire
 		(pts
-			(xy 43.18 180.34) (xy 43.18 172.72)
+			(xy 35.56 180.34) (xy 35.56 172.72)
 		)
 		(stroke
@@
 	(wire
 		(pts
-			(xy 38.1 180.34) (xy 38.1 175.26)
+			(xy 30.48 180.34) (xy 30.48 175.26)
 		)
 		(stroke
@@
 	(wire
 		(pts
-			(xy 26.67 177.8) (xy 33.02 177.8)
+			(xy 19.05 177.8) (xy 25.4 177.8)
 		)
 		(stroke
@@
 	)
 	(label "A2"
-		(at 26.67 177.8 0)
+		(at 19.05 177.8 0)
 		(effects
 			(font
@@
 	)
 	(label "A0"
-		(at 26.67 172.72 0)
+		(at 19.05 172.72 0)
 		(effects
 			(font
@@
 		)
 	)
+	(label "ENC_SW"
+		(at 44.45 176.53 0)
+		(effects
+			(font
+				(size 1.27 1.27)
+			)
+			(justify left bottom)
+		)
+	)
 	(label "A1"
-		(at 26.67 175.26 0)
+		(at 19.05 175.26 0)
 		(effects
 			(font
@@
 	(symbol
 		(lib_id "power:GND")
-		(at 33.02 180.34 0)
+		(at 25.4 180.34 0)
 		(unit 1)
 		(exclude_from_sim no)
@@
 		(fields_autoplaced yes)
 		(property "Reference" "#PWR08"
-			(at 33.02 186.69 0)
+			(at 25.4 186.69 0)
 			(effects
 				(font
@@
 		)
 		(property "Value" "GND"
-			(at 33.02 185.42 0)
+			(at 25.4 185.42 0)
 			(effects
 				(font
@@
 		)
 		(property "Footprint" ""
-			(at 33.02 180.34 0)
+			(at 25.4 180.34 0)
 			(effects
 				(font
@@
 		)
 		(property "Datasheet" ""
-			(at 33.02 180.34 0)
+			(at 25.4 180.34 0)
 			(effects
 				(font
@@
 		)
 		(property "Description" "Power symbol creates a global label with name \"GND\" , ground"
-			(at 33.02 180.34 0)
+			(at 25.4 180.34 0)
 			(effects
 				(font
@@
 	(symbol
 		(lib_id "power:GND")
-		(at 43.18 180.34 0)
+		(at 35.56 180.34 0)
 		(unit 1)
 		(exclude_from_sim no)
@@
 		(fields_autoplaced yes)
 		(property "Reference" "#PWR010"
-			(at 43.18 186.69 0)
+			(at 35.56 186.69 0)
 			(effects
 				(font
@@
 		)
 		(property "Value" "GND"
-			(at 43.18 185.42 0)
+			(at 35.56 185.42 0)
 			(effects
 				(font
@@
 		)
 		(property "Footprint" ""
-			(at 43.18 180.34 0)
+			(at 35.56 180.34 0)
 			(effects
 				(font
@@
 		)
 		(property "Datasheet" ""
-			(at 43.18 180.34 0)
+			(at 35.56 180.34 0)
 			(effects
 				(font
@@
 		)
 		(property "Description" "Power symbol creates a global label with name \"GND\" , ground"
-			(at 43.18 180.34 0)
+			(at 35.56 180.34 0)
 			(effects
 				(font
@@
 	(symbol
 		(lib_id "power:GND")
-		(at 38.1 180.34 0)
+		(at 30.48 180.34 0)
 		(unit 1)
 		(exclude_from_sim no)
@@
 		(fields_autoplaced yes)
 		(property "Reference" "#PWR09"
-			(at 38.1 186.69 0)
+			(at 30.48 186.69 0)
 			(effects
 				(font
@@
 		)
 		(property "Value" "GND"
-			(at 38.1 185.42 0)
+			(at 30.48 185.42 0)
 			(effects
 				(font
@@
 		)
 		(property "Footprint" ""
-			(at 38.1 180.34 0)
+			(at 30.48 180.34 0)
 			(effects
 				(font
@@
 		)
 		(property "Datasheet" ""
-			(at 38.1 180.34 0)
+			(at 30.48 180.34 0)
 			(effects
 				(font
@@
 		)
 		(property "Description" "Power symbol creates a global label with name \"GND\" , ground"
-			(at 38.1 180.34 0)
+			(at 30.48 180.34 0)
 			(effects
 				(font

Commit message: fix: disconnect unused COL5 of switch matrix in favor of encoder switch
Connections:
- no-connect marks 33 -> 34
Changed lines of the file:
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@@
-	)
-	(junction
-		(at 53.34 176.53)
-		(diameter 0)
-		(color 0 0 0 0)
 	)
 	(junction
@@
 	)
 	(no_connect
+		(at 96.52 176.53)
+	)
+	(no_connect
 		(at 167.64 166.37)
 	)
@@
 	(wire
 		(pts
-			(xy 44.45 176.53) (xy 53.34 176.53)
+			(xy 46.99 168.91) (xy 58.42 168.91)
 		)
 		(stroke
@@
 	(wire
 		(pts
-			(xy 53.34 168.91) (xy 58.42 168.91)
-		)
-		(stroke
-			(width 0)
-			(type default)
-		)
-	)
-	(wire
-		(pts
 			(xy 229.87 59.69) (xy 232.41 59.69)
 		)
@@
 	(wire
 		(pts
+			(xy 96.52 176.53) (xy 99.06 176.53)
+		)
+		(stroke
+			(width 0)
+			(type default)
+		)
+	)
+	(wire
+		(pts
 			(xy 72.39 109.22) (xy 74.93 109.22)
 		)
@@
 	(wire
 		(pts
-			(xy 53.34 176.53) (xy 99.06 176.53)
-		)
-		(stroke
-			(width 0)
-			(type default)
-		)
-	)
-	(wire
-		(pts
 			(xy 91.44 119.38) (xy 91.44 124.46)
 		)
@@
 		(pts
 			(xy 72.39 104.14) (xy 86.36 104.14)
-		)
-		(stroke
-			(width 0)
-			(type default)
-		)
-	)
-	(wire
-		(pts
-			(xy 53.34 176.53) (xy 53.34 168.91)
 		)
 		(stroke
@@
 	)
 	(label "ENC_SW"
-		(at 44.45 176.53 0)
-		(effects
-			(font
+		(at 46.99 168.91 0)
+		(effects
+			(font

Commit message: fix: swap 3V3 and GND for SSD1306 Module
Connections:
- net +3.3V: now also J1.2 (Pin_2); no longer J1.1 (Pin_1)
- net GND: now also J1.1 (Pin_1); no longer J1.2 (Pin_2)
Other:
- moved on the sheet: J1
Changed lines of the file:
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@@
 	(wire
 		(pts
-			(xy 121.92 151.13) (xy 121.92 153.67)
+			(xy 121.92 148.59) (xy 121.92 146.05)
 		)
 		(stroke
@@
 	(wire
 		(pts
-			(xy 121.92 148.59) (xy 134.62 148.59)
+			(xy 121.92 151.13) (xy 134.62 151.13)
 		)
 		(stroke
@@
 	(wire
 		(pts
-			(xy 134.62 151.13) (xy 121.92 151.13)
+			(xy 134.62 148.59) (xy 121.92 148.59)
 		)
 		(stroke
@@
 	(wire
 		(pts
-			(xy 134.62 153.67) (xy 125.73 153.67)
+			(xy 134.62 146.05) (xy 125.73 146.05)
 		)
 		(stroke
@@
 	(wire
 		(pts
-			(xy 134.62 156.21) (xy 125.73 156.21)
+			(xy 125.73 143.51) (xy 134.62 143.51)
 		)
 		(stroke
@@
 	(wire
 		(pts
-			(xy 121.92 146.05) (xy 121.92 148.59)
+			(xy 121.92 153.67) (xy 121.92 151.13)
 		)
 		(stroke
@@
 	)
 	(label "I2C0_SCL"
-		(at 125.73 153.67 0)
+		(at 125.73 146.05 0)
 		(effects
 			(font
@@
 	)
 	(label "I2C0_SDA"
-		(at 125.73 156.21 0)
+		(at 125.73 143.51 0)
 		(effects
 			(font
@@
 		(lib_id "power:+3V3")
 		(at 121.92 146.05 0)
+		(mirror y)
 		(unit 1)
 		(exclude_from_sim no)
@@
 	(symbol
 		(lib_id "Connector:Conn_01x04_Socket")
-		(at 139.7 151.13 0)
+		(at 139.7 148.59 0)
+		(mirror x)
 		(unit 1)
 		(exclude_from_sim no)
@@
 		(dnp no)
 		(property "Reference" "J1"
-			(at 140.97 151.1299 0)
+			(at 140.97 148.5901 0)
 			(effects
 				(font
@@
 		)
 		(property "Value" "SSD1306 Module"
-			(at 124.714 143.51 0)
+			(at 123.698 154.178 0)
 			(effects
 				(font
@@
 		)
 		(property "Footprint" "spur-demo:SSD1306"
-			(at 139.7 151.13 0)
+			(at 139.7 148.59 0)
 			(effects
 				(font
@@
 		)
 		(property "Datasheet" "~"
-			(at 139.7 151.13 0)
+			(at 139.7 148.59 0)
 			(effects
 				(font
@@
 		)
 		(property "Description" "Generic connector, single row, 01x04, script generated"
-			(at 139.7 151.13 0)
+			(at 139.7 148.59 0)
 			(effects
 				(font
@@
 		(lib_id "power:GND")
 		(at 121.92 153.67 0)
+		(mirror y)
 		(unit 1)
 		(exclude_from_sim no)

Commit message: fix: correct pulldown resistor values from values used in pullup configuration
Parts:
- R26, R27: value 56k -> 5.1k
Changed lines of the file:
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@@
 			)
 		)
-		(property "Value" "56k"
+		(property "Value" "5.1k"
 			(at 52.07 64.7699 0)
 			(effects
@@
 			)
 		)
-		(property "Value" "56k"
+		(property "Value" "5.1k"
 			(at 41.91 64.7699 0)
 			(effects

Commit message: fix: update PCB to reflect corrected NTC network, reroute
Other:
- note added: "USB Interface USB 2.0 @ 500 mA"
- note removed: "USB Interface On-The-Go @ 500 mA"
- moved on the sheet: SW23
