File: Hardware/KiCAD/spur-demo/spur-demo.kicad_pcb (KiCad board)
At the start: 2 copper layers, 63.8 x 105.5 mm, 74 parts, among them IC1 BQ24193RGER, IC2 PCF8575PWR, IC3 ISL91127IRNZ-T7A, J1 SSD1306 Module, J12 USB_C_Plug_USB2.0, J2 Conn_Coaxial, J4 VMA309 Module, J5 Conn_01x02, J6 Conn_01x08_Socket, J7 PAM8392A Module, J8 1x15, J9 1x15, Q1 ZXMN2A01F, U1 SA868, U4 LM393, U5 XCVR_ESP32-C3-DEVKITM-1

Commit message: feat: completely reroute demo PCB, zones still not fully connected
Parts:
- moved R20 63.1 mm to (36.9, 115.8), turned to 0 degrees
- moved R22 62.1 mm to (40.9, 120.1), turned to -90 degrees
- moved R23 59.9 mm to (42.4, 120.1), turned to -90 degrees
- moved R12 58.3 mm to (53.8, 114.0), turned to 90 degrees
- moved MK1 0.18 mm to (82.9, 93.3)
- moved J2 0.07 mm to (40.8, 49.0)
Routing:
- net /VOL: track 0.01 -> 123.8 mm, vias 0 -> 2
- net /RADIO_TXD: track 0.01 -> 84.8 mm
- net +3.3V: track 226.6 -> 301.3 mm
- net /AMP_BCLK: track 75.9 -> 2.69 mm, vias 2 -> 0
- net /Computing Subsystem/SPIM2_MISO: track 76.2 -> 6.98 mm, vias 1 -> 0
- net /~{BMS_CE}: track 3.25 -> 64.4 mm, vias 0 -> 2
- net GND: track 104.6 -> 55.7 mm, vias 8 -> 24
- net /RADIO_RXD: track 46.9 -> 88.7 mm
- net Net-(IC3-PVIN_1): track 99.7 -> 138.0 mm
- net /~{SPIM2_CS}: track 37.0 -> 0.00 mm, vias 2 -> 0
- net /~{AMP_SD}: track 68.9 -> 37.6 mm, vias 2 -> 0
- net /I2C0_SCL: track 149.2 -> 179.2 mm
- net /I2C0_SDA: track 152.3 -> 175.0 mm, vias 5 -> 6
- net /Keypad/COL4: track 35.9 -> 19.0 mm
- net /Keypad/COL1: track 23.2 -> 39.2 mm
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Other:
- outline, holes or cut-outs redrawn

Commit message: feat: finish DRC of demo PCB and remove islanding
Routing:
- net +3.3V: track 301.3 -> 271.7 mm, vias 2 -> 3
- net /BMS_INT: track 63.3 -> 75.0 mm
- net /VOL: track 123.8 -> 113.9 mm, vias 2 -> 0
- net Net-(IC3-PVIN_1): track 138.0 -> 131.1 mm
- net /Keypad/COL1: track 39.2 -> 35.8 mm
- net /Keypad/COL2: track 34.0 -> 31.1 mm
- net /I2C0_SDA: track 175.0 -> 172.3 mm, vias 6 -> 5
- net /~{Audio_ON}: track 59.4 -> 61.6 mm
- net /Keypad/COL3: track 28.7 -> 26.5 mm
- net /I2C0_SCL: track 179.2 -> 179.8 mm
- net /RADIO_RXD: track 88.7 -> 89.3 mm
- net GND: track 55.7 -> 55.5 mm, vias 24 -> 140

Commit message: feat: add rotary encoder to demo board
Parts:
- added SW23: RotaryEncoder_Switch, Rotary_Encoder:RotaryEncoder_Bourns_Horizontal_PEC12R-2x17F-Sxxxx, F.Cu at (57.6, 47.8)
- moved J1 7.42 mm to (70.0, 53.6)
Connections:
- IC2 pad 4: /~{BMS_CE} -> /ENC_CLK
- IC2 pad 5: unconnected-(IC2-P01-Pad5) -> /ENC_DT
- IC2 pad 7: /OLED_D/~{C} -> /~{BMS_CE}
Routing:
- net /ENC_DT: track 0.00 -> 98.7 mm, vias 0 -> 1
- net /ENC_CLK: track 0.00 -> 95.2 mm, vias 0 -> 1
- net /I2C0_SCL: track 179.8 -> 172.7 mm
- net /I2C0_SDA: track 172.3 -> 165.3 mm
- net +3.3V: track 271.7 -> 275.1 mm
- net GND: track 55.5 -> 54.0 mm, vias 140 -> 146

Commit message: chore: specify encoder footprint, replot demo schematic
Parts:
- SW23: moved to B.Cu
- moved SW23 5.00 mm to (52.6, 47.7)
Routing:
- net /ENC_CLK: track 95.2 -> 99.9 mm
- net /ENC_DT: track 98.7 -> 96.0 mm, vias 1 -> 3
- net /~{BMS_CE}: track 64.4 -> 66.2 mm

Commit message: fix: disconnect unused COL5 of switch matrix in favor of encoder switch
Connections:
- IC2 pad 11: /Keypad/COL5 -> /ENC_SW
Routing:
- net /ENC_SW: track 0.00 -> 100.0 mm, vias 0 -> 1
- net /ENC_CLK: track 99.9 -> 100.4 mm
- net GND: vias 146 -> 148

Commit message: fix: swap 3V3 and GND for SSD1306 Module
Connections:
- J1 pad 1: +3.3V -> GND
- J1 pad 2: GND -> +3.3V
Routing:
- net +3.3V: track 275.4 -> 276.4 mm

Commit message: fix: update PCB to reflect corrected NTC network, reroute
Parts:
- H1, H2: value MountingHole_2.2mm_M2_Pad_Via -> MountingHole_2.7mm_M2_Pad_Via; footprint MountingHole:MountingHole_2.2mm_M2_Pad_Via -> MountingHole:MountingHole_2.7mm_Pad_Via
- R26, R27: value 56k -> 5.1k
- moved JP7 11.9 mm to (86.3, 116.4), turned to -90 degrees
- moved R1 7.16 mm to (85.7, 130.7)
- moved JP11 4.38 mm to (85.2, 127.4), turned to 180 degrees
- moved TH1 2.54 mm to (66.0, 130.8), turned to 180 degrees
- moved H2 1.87 mm to (90.5, 139.7)
- moved H1 0.76 mm to (66.8, 139.7)
Connections:
- IC1 pad 11: /Power Subsystem/TS_P -> Net-(IC1-TS1)
- IC1 pad 12: /Power Subsystem/TS_P -> Net-(IC1-TS1)
- R2 pad 1: /Power Subsystem/TS_N -> Net-(IC1-TS1)
- R3 pad 2: /Power Subsystem/TS_N -> Net-(IC1-TS1)
- TH1 pad 1: /Power Subsystem/TS_N -> GND
- TH1 pad 2: /Power Subsystem/TS_P -> Net-(IC1-TS1)
Routing:
- net Net-(IC1-TS1): track 0.00 -> 46.4 mm, vias 0 -> 1
- net /Power Subsystem/TS_N: track 32.3 -> 0.00 mm, vias 1 -> 0
- net /Power Subsystem/TS_P: track 20.7 -> 0.00 mm, vias 1 -> 0
- net +3.3V: track 276.4 -> 294.4 mm
- net Net-(IC1-PSEL): track 21.4 -> 14.2 mm
- net +SYS: track 127.5 -> 122.1 mm
- net /BMS_INT: track 75.0 -> 69.8 mm
- net /BMS_OTG: track 12.3 -> 16.7 mm
- net /ENC_SW: track 100.0 -> 96.5 mm
- net /~{BMS_CE}: track 66.2 -> 63.7 mm
- net VBUS: track 42.8 -> 45.0 mm
- net +BATT: track 34.3 -> 32.2 mm
- net /I2C0_SDA: track 165.3 -> 163.2 mm
- net /ENC_CLK: track 100.4 -> 98.5 mm
- net /MIC_IN: track 67.4 -> 68.4 mm
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Other:
- board text added: "3V3 GND TOOL0 NRST"
- board text added: "Eric Mutton KJ5DIF ECE 4V97 Rev. B"
- board text added: "OTG"
- board text added: "PG"
- board text added: "PSEL"
- board text added: "RL78"
- board text added: "STAT"
