File: Hardware/KiCAD/bms-smps-testbench/bms-smps-testbench.kicad_pcb (KiCad board)
At the start: 2 copper layers, 50.8 x 32 mm, 32 parts, among them IC1 BQ24193RGER, IC3 ISL91127IRNZ-T7A, J1 Screw_Terminal_01x02, J2 Screw_Terminal_01x02, J3 Screw_Terminal_01x02, J4 Screw_Terminal_01x02, J5 Screw_Terminal_01x05, J6 USB_A

Commit message: chore: plot schematic and update to KiCAD 9.0, export 3D image
Parts:
- TH1: moved to F.Cu
- turned TH1 to 90 degrees
