File: Hardware/KiCAD/bms-smps-testbench/bms-smps-testbench.kicad_sch (KiCad schematic)
At the start: 37 parts, among them IC1 BQ24193RGER, IC2 TPS61235PRWLT, IC3 ISL91127IRNZ-T7A, J1 Screw_Terminal_01x02, J2 Screw_Terminal_01x02, J3 Screw_Terminal_01x02, J4 Screw_Terminal_01x02, J5 Screw_Terminal_01x05, J6 USB_A, U1 BQ297xy

Commit message: fix: bring sa8x8 flexypins closer, add smps resistor
Parts:
- added R1: 2.2M, Resistor_SMD:R_0603_1608Metric, symbol Device:R_US
- R11: value 2.2M -> 1M
Connections:
- net GND: now also R1.2; no longer R11.2
- new net: R1.1, R11.2
Other:
- note added: "I_{INMAX} = (1V / R8) × 530 Typical I_{INMAX} = (1V / 265R) × 530 = 2A Common I_{INMAX} = (1V / 267R) × 530 = 1.99A Placed R8: 267R"
- note added: "V_{OUT} = 0.8V * (1 + R1/R2) (3.3V)/0.8 - 1 = R1/R2 For C3 = 56p, R1 = 1M R2 = R1*3.125 = 3.125M Common values: 2.2M + 1M (-1.12%)"
- note removed: "V_{OUT} = 0.8V * (1 + R1/R2) (3.3V)/0.8 - 1 = R1/R2 For R3 = 56p, R1 = 1M R2 = R1*3.125 = 3.125M Common values: 2.2M + 1M (-1.12%)"
Changed lines of the file:
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@@
 	(wire
 		(pts
-			(xy 252.73 153.67) (xy 237.49 153.67)
+			(xy 237.49 153.67) (xy 242.57 153.67)
 		)
 		(stroke
@@
 	(wire
 		(pts
+			(xy 250.19 153.67) (xy 252.73 153.67)
+		)
+		(stroke
+			(width 0)
+			(type default)
+		)
+	)
+	(wire
+		(pts
 			(xy 46.99 137.16) (xy 49.53 137.16)
 		)
@@
 	(wire
 		(pts
-			(xy 252.73 151.13) (xy 252.73 153.67)
-		)
-		(stroke
-			(width 0)
-			(type default)
-		)
-	)
-	(wire
-		(pts
 			(xy 67.31 154.94) (xy 67.31 162.56)
 		)
@@
 	(wire
 		(pts
+			(xy 252.73 153.67) (xy 252.73 151.13)
+		)
+		(stroke
+			(width 0)
+			(type default)
+		)
+	)
+	(wire
+		(pts
 			(xy 143.51 29.21) (xy 146.05 29.21)
 		)
@@
 		)
 	)
+	(text "\nI_{INMAX} = (1V / R8) × 530\nTypical I_{INMAX} = (1V / 265R) × 530 = 2A\nCommon I_{INMAX} = (1V / 267R) × 530 = 1.99A\n\nPlaced R8: 267R"
+		(exclude_from_sim no)
+		(at 56.642 82.804 0)
+		(effects
+			(font
+				(size 1.27 1.27)
+			)
+			(justify left)
+		)
+	)
 	(text "BMS Single-Cell"
 		(exclude_from_sim no)
@@
 		)
 	)
-	(text "V_{OUT} = 0.8V * (1 + R1/R2)\n(3.3V)/0.8 - 1 = R1/R2\n\nFor R3 = 56p, R1 = 1M\nR2 = R1*3.125 = 3.125M\n\nCommon values:\n2.2M + 1M (-1.12%)"
+	(text "V_{OUT} = 0.8V * (1 + R1/R2)\n(3.3V)/0.8 - 1 = R1/R2\n\nFor C3 = 56p, R1 = 1M\nR2 = R1*3.125 = 3.125M\n\nCommon values:\n2.2M + 1M (-1.12%)"
 		(exclude_from_sim no)
 		(at 245.872 73.152 0)
@@
 	)
 	(symbol
+		(lib_id "Device:R_US")
+		(at 246.38 153.67 270)
+		(unit 1)
+		(exclude_from_sim no)
+		(in_bom yes)
+		(on_board yes)
+		(dnp no)
+		(fields_autoplaced yes)
+		(property "Reference" "R1"
+			(at 246.38 147.32 90)
+			(effects
+				(font
+					(size 1.27 1.27)
+				)
+			)
+		)
+		(property "Value" "2.2M"
+			(at 246.38 149.86 90)
+			(effects
+				(font
+					(size 1.27 1.27)
+				)
+			)
+		)
+		(property "Footprint" "Resistor_SMD:R_0603_1608Metric"
+			(at 246.126 154.686 90)
+			(effects
+				(font
+					(size 1.27 1.27)
+				)
+				(hide yes)
+			)
+		)
+		(property "Datasheet" "~"
+			(at 246.38 153.67 0)
+			(effects
+				(font
+					(size 1.27 1.27)
+				)
+				(hide yes)
+			)
+		)
+		(property "Description" "Resistor, US symbol"
+			(at 246.38 153.67 0)
+			(effects
+				(font
+					(size 1.27 1.27)
+				)
+				(hide yes)
+			)
+		)
+		(pin "1"
+		)
+		(pin "2"
+		)
+		(instances
+			(project "bms-smps-testbench"
+				(path "/b2964315-5f76-41bb-a1d4-04083937cdc0"
+					(reference "R1")
+					(unit 1)
+				)
+			)
+		)
+	)
+	(symbol
 		(lib_id "Cobalt-Cowboy:TPS61235PRWLT")
 		(at 208.28 59.69 0)
@@
 			)
 		)
-		(property "Value" "2.2M"
+		(property "Value" "1M"
 			(at 255.27 148.5899 0)
 			(effects
